File: CameraBoard/eagle/CameraBoard.sch (EAGLE design)
At the start: 11 parts

Commit message: adding first design review notes
Parts:
- added C10, C5, C6: 10u, oresat-rcl:C-EU0805-C-NOSILK
- added C28, C8, C9: 22u, oresat-rcl:C-EU0805-C-NOSILK
- added C7: 100n, oresat-rcl:C-EU0603-C-NOSILK
- added JP12: (no value), pinhead:PINHD-1X2
- added L1: 1.5uH, L--IHLP2020CZER1R5M11--1.5uHInductor:IHLP2020CZER1R5M11
- added R1, R4: 10k, oresat-rcl:R-US_0603-C-NOSILK
- added R2: 470k, oresat-rcl:R-US_0603-C-NOSILK
- added R3: 150k, oresat-rcl:R-US_0603-C-NOSILK
- added TP26, TP27, TP28, TP29, TP6: TEST-POINT, Tova:TEST-POINT
- added U10: TPS63070, ic-pwr-tps63070x:TPS63070X
- JP10: device pinhead:PINHD-1X2 -> pinhead:PINHD-1X4
Connections:
- new net +12V: C10.1, C5.1, C6.1, R1.2, U10.VIN
- new net 3.3V: C28.1, C8.1, C9.1, R2.2, TP6.1, U10.VOUT
- new net TPS-EN: R1.1, TP29.1, U10.EN, U10.PS/SYNC
- new net TPS-FB: R2.1, R3.2, U10.FB
- new net TPS-FB2: TP27.1, U10.FB2
- new net TPS-L1: L1.P$1, U10.L1
- new net TPS-L2: L1.P$2, U10.L2
- new net TPS-PG: TP26.1, U10.PG
- new net TPS-VAUX: C7.1, U10.VAUX
- new net TPS-VSEL: R4.2, TP28.1, U10.VSEL
- net GND: now also C10.2, C28.2, C5.2, C6.2, C7.2, C8.2, C9.2, R3.1, R4.1, U10.GND, U10.PGND
Other:
- note added: "0805"
- note added: "Power Switch"

Commit message: power schematic for board
Parts:
- removed U10: TPS63070, ic-pwr-tps63070x:TPS63070X
- added C1: 4.7u, oresat-rcl:C-EU0603-A-NOSILK
- added C11: 2.2n, oresat-rcl:C-EU0603-A-NOSILK
- added C12, C2: 0.1u, oresat-rcl:C-EU0603-A-NOSILK
- added C13: 1u, oresat-rcl:C-EU0603-A-NOSILK
- added C14: 0.01u, oresat-rcl:C-EU0603-A-NOSILK
- added C15, C16, C17, C18: 10u, oresat-rcl:C-EU0603-C-NOSILK
- added C19, C20, C21: 47u, oresat-rcl:C-EU1206-A
- added C3: 10u, oresat-rcl:C-EU0603-A-NOSILK
- added C4: 4.7n, oresat-rcl:C-EU0603-A-NOSILK
- added D1, D3, D4: SML-D12U1WT86, led:LEDCHIPLED_0603
- added D2, D5, D6: D_MBRS340T3G, D--MBRS340T3G--Schottky Diode:D_MBRS340T3G
- added L2: 1239AS-H-100M=P2, L--1239AS-H-100M=P2--10uH Inductor:1239AS-H-100M=P2
- added L3: 22u, oresat-rcl:L-US0805-C-NOSILK
- added Q1: SI7465DP-T1-E3, Q--Si7465DP--Vishay Power MOSFET with multple S+D leads:SI7465DP-T1-E3
- added R10: 750, oresat-rcl:R-US_0603-A-NOSILK
- added R11: 200m, oresat-rcl:R-US_0603-A-NOSILK
- added R12: 10K, R--NHQ103B375T10--Thermistor 10K:NHQ103B375T10
- added R13, R14, R15: 1k, oresat-rcl:R-US_0603-A-NOSILK
- added R5: 221, oresat-rcl:R-US_0603-C-NOSILK
- added R6, R7: 230, oresat-rcl:R-US_0603-A-NOSILK
- added R8: 10k, oresat-rcl:R-US_0603-A-NOSILK
- added R9: 42.5k, oresat-rcl:R-US_0603-A-NOSILK
- added U1: MP26124GR-Z, U--MP26124GR-Z--4S LiPo Charger :MP26124GR-Z
- added U2: TPS63070, ic-pwr-tps63070x:TPS63070X
- added U3: LM2678SD-12/NOPB, U--LM2678SX-12-NOPB--TI 12V SPS:LM2678SD-12/NOPB
- JP11: device pinhead:PINHD-1X4 -> pinhead:PINHD-1X6
- R2: value 470k -> 680k
- R3: value 150k -> 130k
Connections:
- removed net 3.3V: C28.1, C8.1, C9.1, R2.2, TP6.1, U10.VOUT
- new net +16V: C15.1, C16.1, C17.1, C18.1, Q1.D, U3.IN
- new net +5V: C28.1, C8.1, C9.1, D1.A, JP12.1, R2.2, TP6.1, U2.VOUT
- new net ARM-IN: JP11.6, R14.2
- new net ARM-OUT: JP11.5, R15.1
- new net CHUTE: JP11.2
- new net DROGUE: JP11.3
- new net N$1: D1.C, R5.2
- new net N$10: R12.P$1, R8.1, U1.NTC
- new net N$11: R9.1, U1.COMPV
- new net N$12: C11.1, R9.2
- new net N$13: R10.1, U1.COMPI
- new net N$14: C4.1, R10.2
- new net N$15: C2.1, D5.-, L2.P$1, U1.SW
- new net N$16: C2.2, U1.BST
- new net N$17: L2.P$2, R11.1, U1.CSP
- new net N$18: C14.1, D6.-, L3.1, U3.SOUT
- new net N$2: C1.1, D2.-, U1.VIN
- new net N$20: C14.2, U3.CB
- new net N$3: Q1.G, R13.2, R14.1
- new net N$4: C13.1, R6.2, R7.2, R8.2, U1.VREF33
- new net N$5: D4.A, R6.1
- new net N$6: D3.A, R7.1
- new net N$7: D3.C, U1.!CHGOK
- new net N$8: D4.C, U1.!ACOK
- new net N$9: C12.1, U1.TMR
- new net TGND: JP11.1
- new net VUMB: D2.+, JP11.4, U1.VCC
- net +12V: now also C19.1, C20.1, C21.1, L3.2, U2.VIN, U3.FB; no longer U10.VIN
- net BATT+: now also C3.1, JP10.1, JP10.2, Q1.S, R11.2, R15.2, U1.BATT
- net GND: now also C1.2, C11.2, C12.2, C13.2, C15.2, C16.2, C17.2, C18.2, C19.2, C20.2, C21.2, C3.2, C4.2, D5.+, D6.+, JP10.3, JP10.4, JP12.2, R12.P$2, R13.1, U1.!EN, U1.GND, U1.SGND, U2.GND, U2.PGND, U3.GND; no longer U10.GND, U10.PGND
- net TPS-EN: now also U2.EN, U2.PS/SYNC; no longer U10.EN, U10.PS/SYNC
- net TPS-FB: now also U2.FB; no longer U10.FB
- net TPS-FB2: now also U2.FB2; no longer U10.FB2
- net TPS-L1: now also U2.L1; no longer U10.L1
- net TPS-L2: now also U2.L2; no longer U10.L2
- net TPS-PG: now also U2.PG; no longer U10.PG
- net TPS-VAUX: now also U2.VAUX; no longer U10.VAUX
- net TPS-VSEL: now also U2.VSEL; no longer U10.VSEL
Other:
- note added: "12V to 5V SPS"
- note added: "16.8V to 12V SPS"
- note added: "ARM+ ARM- VUMB DROGUE CHUTE TGND"
- note added: "Arming Switch"
- note added: "Comp selection: -Datasheet called for polarized -The diode has 4A rating"
- note added: "Incoming signals"
- note added: "Keep feedback wire away from inductor flux on board"
- note added: "LED to indicate power is on"
- note added: "LiPo Charger"
- note added: "Power to ATV Transmitter"
- note added: "Usually on unless Arm-In and Arm-Out are shorted"
- note removed: "Power Switch"
- note removed: "The Charger"
- moved on the sheet: C10, C28, C5, C6, C7, C8, C9, JP10, JP12, L1, R1, R2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

Commit message: first draft of schematic complete
Parts:
- added C22: 1u, oresat-rcl:C-EU0603-C-NOSILK
- added C23: 20u, oresat-rcl:C-EU0603-C-NOSILK
- added Q2: BVSS123LT1G, Q--BVSS123LT1G--NCH MOSFET:BVSS123LT1G
- added Q3: BSS84, Q--BSS84CT-ND--PCH MOSFET:BSS84
- added R16: 237k, oresat-rcl:R-US_0603-A-NOSILK
- added R17, R28: 10k, oresat-rcl:R-US_0603-C-NOSILK
- added R18, R19: 60.4, oresat-rcl:R-US_0603-C-NOSILK
- added R20, R21: 10k, oresat-rcl:R-US_0603-A-NOSILK
- added R22: 1k, oresat-rcl:R-US_0603-A-NOSILK
- added R23: 10, oresat-rcl:R-US_0603-A-NOSILK
- added U4: TS5A3159ADBVR, U--TS5A3159ADBVR--Analog Switch 5V and 3V3:TS5A3159ADBVR
- added U5: ICM7242IBAZ-SMD, U--ICM7242--Counter-Timer Circuit:ICM7242IBAZ-SMD
- added U6, U7: H11F1SR2M, Q--H11F1SR2M--OptoIsolator:H11F1SR2M
- added U8: SN74LVC1G17DCKR, U--SN74LVC1G17--Schmitt Trigger Buffer:SN74LVC1G17DCKR
- JP12: device pinhead:PINHD-1X2 -> pinhead:PINHD-1X4
Connections:
- removed net TGND: JP11.1
- new net CAM_DOWN: JP9.3, U4.NO
- new net CAM_UP: JP8.3, U4.NC
- new net N$22: R18.1, U6.CAT
- new net N$23: R19.1, U7.CAT
- new net N$24: C22.1, R16.2, U5.RC
- new net N$25: C23.1, Q2.D, Q3.D
- new net N$26: Q3.S, R23.2
- new net N$28: Q3.G, R20.1
- new net N$29: Q2.G, R21.1
- new net SCHMITTIN: Q2.S, R22.1, U8.A
- new net TIMERPULSE: R17.1, R20.2, R21.2, R28.1, U6.OUT, U7.OUT
- new net TIMER_OUTPUT: U4.IN, U5./128, U5.RESET
- new net TIMER_TRIGG: U5.TRIGGER, U8.Y
- new net T_GND: JP11.1, R18.2, R19.2
- new net VIDEO_OUT: JP12.3, U4.COM
- net +12V: now also JP1.1, JP2.1, JP3.1, JP4.1, JP5.1, JP6.1, JP7.1, JP8.1, JP9.1
- net +5V: now also C22.2, R16.1, R23.1, U4.V+, U5.VDD, U6.IN, U7.IN, U8.VCC
- net BATT+: no longer JP1.1, JP2.1, JP3.1, JP4.1, JP5.1, JP6.1, JP7.1, JP8.1, JP9.1
- net CHUTE: now also U7.ANOD
- net DROGUE: now also U6.ANOD
- net GND: now also C23.2, R17.2, R22.2, R28.2, U4.GND, U5.VSS, U8.GND
Other:
- note added: "A high signal from either drogue or main will tell the pulse generator to send the timer a pulse"
- note added: "Camera Operation"
- note added: "Cameras"
- note added: "Input Signals"
- note added: "Pulse Generator"
- note added: "This generates a 0.02 second pulse when TIMERPULSE is high"
- note added: "This timer is in monostable mode, so connect time output to the reset"
- note added: "Timer"
- note added: "When TIMER_OUTPUT is high, switches to the normally closed input as video transmission"
- note removed: "The Cameras"
- moved on the sheet: JP1, JP2, JP3, JP4, JP5, JP6, JP7, JP8, JP9, U3

Commit message: layed out board before routing
Parts:
- added C24: 0.1u, oresat-rcl:C-EU0603-C-NOSILK
- C15, C16, C17, C18: device oresat-rcl:C-EU0603-C-NOSILK -> oresat-rcl:C-EU0805-B-NOSILK
- L3: value 22u -> 784770220; device oresat-rcl:L-US0805-C-NOSILK -> L--784770220--22uH 4A Inductor:784770220
Connections:
- net TIMER_OUTPUT renamed !TIMER_OUTPUT
- removed net N$18: C14.1, D6.-, L3.1, U3.SOUT
- new net 12V_OUT: C14.1, D6.-, L3.P$1, U3.SOUT
- net +12V: now also L3.P$2; no longer L3.2
- net +5V: now also C24.1
- net GND: now also C24.2
Other:
- note added: "This timer is in monostable mode, so TIMER_OUTPUT is connected to the reset"
- note added: "When IN is HIGH, NO connects to COM"
- note added: "When TIMER_OUTPUT is low, switches to the normally closed input as video transmission"
- note removed: "This timer is in monostable mode, so connect time output to the reset"
- note removed: "When TIMER_OUTPUT is high, switches to the normally closed input as video transmission"
- moved on the sheet: C22, C23, JP1, JP2, JP3, JP4, JP5, JP6, JP7, JP8, JP9, R16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

Commit message: finished board layout before routing
Parts:
- renumbered JP10 to BATTERY, JP11 to INPUTS, JP12 to ATV, JP8 to CAM_UP, JP9 to CAM_DOWN

Commit message: completed routing of board rev 1.0
Parts:
- D2, D5: value D_MBRS340T3G -> S2MA-13-F; device D--MBRS340T3G--Schottky Diode:D_MBRS340T3G -> D--S2MA-FDICT-ND--Schottky Diode 1.5A:S2MA-13-F
Changed lines of the file:
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@@
 <part name="GND1" library="supply1" deviceset="GND" device=""/>
 <part name="U1" library="U--MP26124GR-Z--4S LiPo Charger " deviceset="MP26124GR-Z" device=""/>
-<part name="D2" library="D--MBRS340T3G--Schottky Diode" deviceset="D_MBRS340T3G" device=""/>
+<part name="D2" library="D--S2MA-FDICT-ND--Schottky Diode 1.5A" deviceset="S2MA-13-F" device=""/>
 <part name="C1" library="oresat-rcl" deviceset="C-EU" device="0603-A-NOSILK" value="4.7u"/>
 <part name="C2" library="oresat-rcl" deviceset="C-EU" device="0603-A-NOSILK" value="0.1u"/>
@@
 <part name="GND10" library="supply1" deviceset="GND" device=""/>
 <part name="L2" library="L--1239AS-H-100M=P2--10uH Inductor" deviceset="1239AS-H-100M=P2" device=""/>
-<part name="D5" library="D--MBRS340T3G--Schottky Diode" deviceset="D_MBRS340T3G" device=""/>
+<part name="D5" library="D--S2MA-FDICT-ND--Schottky Diode 1.5A" deviceset="S2MA-13-F" device=""/>
 <part name="GND11" library="supply1" deviceset="GND" device=""/>
 <part name="R12" library="R--NHQ103B375T10--Thermistor 10K" deviceset="NHQ103B375T10" device="" value="10K"/>
@@
 <attribute name="VALUE" x="124.46" y="78.105" size="1.778" layer="96" rot="R90"/>
 </instance>
-<instance part="D2" gate="A" x="102.87" y="124.46" smashed="yes">
+<instance part="D2" gate="G$1" x="102.87" y="124.46" smashed="yes">
 <attribute name="NAME" x="101.85168125" y="118.746940625" size="1.779809375" layer="95"/>
 </instance>
@@
 <attribute name="NAME" x="160.02" y="104.14" size="1.778" layer="95" font="vector"/>
 </instance>
-<instance part="D5" gate="A" x="153.67" y="97.79" smashed="yes" rot="R90">
+<instance part="D5" gate="G$1" x="153.67" y="97.79" smashed="yes" rot="R90">
 <attribute name="NAME" x="160.40331875" y="97.788059375" size="1.779809375" layer="95" rot="R180"/>
 </instance>
@@
 <segment>
 <pinref part="GND11" gate="1" pin="GND"/>
-<pinref part="D5" gate="A" pin="+"/>
+<pinref part="D5" gate="G$1" pin="+"/>
 </segment>
 <segment>
@@
 <net name="N$2" class="0">
 <segment>
-<pinref part="D2" gate="A" pin="-"/>
+<pinref part="D2" gate="G$1" pin="-"/>
 <pinref part="U1" gate="G$1" pin="VIN"/>
 <wire x1="106.68" y1="124.46" x2="124.46" y2="124.46" width="0.1524" layer="91"/>
@@
 <net name="VUMB" class="0">
 <segment>
-<pinref part="D2" gate="A" pin="+"/>
+<pinref part="D2" gate="G$1" pin="+"/>
 <wire x1="99.06" y1="124.46" x2="97.79" y2="124.46" width="0.1524" layer="91"/>
 <pinref part="U1" gate="G$1" pin="VCC"/>
@@
 <net name="N$15" class="0">
 <segment>
-<pinref part="D5" gate="A" pin="-"/>
+<pinref part="D5" gate="G$1" pin="-"/>
 <pinref part="L2" gate="G$1" pin="P$1"/>
 <pinref part="U1" gate="G$1" pin="SW"/>

Commit message: new image
Connections:
- net GND: now also R5.1
Changed lines of the file:
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@@
 <attribute name="VALUE" x="397.002" y="73.025" size="1.778" layer="96" rot="R90"/>
 </instance>
-<instance part="GND1" gate="1" x="393.7" y="69.85" smashed="yes" rot="MR0">
-<attribute name="VALUE" x="396.24" y="67.31" size="1.778" layer="96" rot="MR0"/>
+<instance part="GND1" gate="1" x="393.7" y="67.31" smashed="yes" rot="MR0">
+<attribute name="VALUE" x="396.24" y="64.77" size="1.778" layer="96" rot="MR0"/>
 </instance>
 <instance part="U1" gate="G$1" x="124.46" y="88.265" smashed="yes">
@@
 <wire x1="396.875" y1="200.66" x2="396.875" y2="203.835" width="0.1524" layer="91"/>
 </segment>
+<segment>
+<pinref part="GND1" gate="1" pin="GND"/>
+<pinref part="R5" gate="R" pin="1"/>
+<wire x1="393.7" y1="69.85" x2="393.7" y2="71.755" width="0.1524" layer="91"/>
+</segment>
 </net>

Commit message: added all the suggestions from first design review
Parts:
- removed ATV, BATTERY: (no value), pinhead:PINHD-1X4
- added C25, C26: 100n, oresat-rcl:C-EU0603-C-NOSILK
- added JP10: (no value), pinhead:PINHD-1X3
- added JP11: (no value), pinhead:PINHD-1X6
- added JP8: (no value), pinhead:PINHD-1X2
- added TP1, TP10, TP11, TP12, TP13, TP14, TP2, TP5, TP7, TP8, TP9: TEST-POINT, Tova:TEST-POINT
- C12, C2, C24: value 0.1u -> 100n
- C14: value 0.01u -> 10n
- L2: value 1239AS-H-100M=P2 -> 10uH
- R11: device oresat-rcl:R-US_0603-A-NOSILK -> oresat-rcl:R-US_1206-A
- R13: value 1k -> 10k
- R23: device oresat-rcl:R-US_0603-A-NOSILK -> oresat-rcl:R-US_0805-A-NOSILK
- R5: value 221 -> 400
- renumbered CAM_DOWN to JP12, CAM_UP to JP13, INPUTS to JP9
Connections:
- net 12V_OUT renamed SOUT
- new net N$18: TP1.1, U3.ON
- net !TIMER_OUTPUT: now also TP9.1
- net +12V: now also TP2.1
- net +5V: now also C25.2, C26.2, JP10.1; no longer ATV.1
- net BATT+: now also JP11.1, JP11.2, JP11.3; no longer BATTERY.1, BATTERY.2
- net CAM_DOWN: now also TP11.1
- net CAM_UP: now also TP12.1
- net CHUTE: now also TP14.1
- net DROGUE: now also TP13.1
- net GND: now also C25.1, C26.1, JP10.2, JP11.4, JP11.5, JP11.6, JP8.2; no longer ATV.2, BATTERY.3, BATTERY.4
- net N$10: now also JP8.1
- net SCHMITTIN: now also TP7.1
- net TIMERPULSE: now also TP5.1
- net TIMER_TRIGG: now also TP8.1
- net VIDEO_OUT: now also JP10.3, TP10.1; no longer ATV.3
Other:
- note added: "All resistors are 1% 0603 packages unless otherwise specified All capacitors are 10% 0603 packages unless otherwise specified"
- note added: "Incoming signals VUMB - 19V"
- note added: "Output: 12V, 5A Max"
- note added: "Output: 16.8V, 1A Max"
- note added: "Output: 5V, 2A Max"
- note added: "Thermistor to be placed on battery through the jumper"
- note added: "This generates a 20ms pulse when TIMERPULSE is high"
- note added: "Timer outputs high for 30seconds when recieving a trigger"
- note removed: "Incoming signals"
- note removed: "This generates a 0.02 second pulse when TIMERPULSE is high"
- moved on the sheet: R12, U1, U3
