File: CameraBoard/kicad/CameraBoard.kicad_sch (KiCad schematic)
At the start: 57 parts, among them Q1 SUD08P06-155L, Q2 SUD08P06-155L, Q3 SUD08P06-155L, U2 MP2659GQ-0000-Z

Commit message: Small BOM changes
Parts:
- C1, C3, C4, C5: DIS (none) -> DigiKey; DPN (none) -> 490-GRT21BC71E106KE13KCT-ND; MPN (none) -> GRT21BC71E106KE13K; Manufacturer (none) -> Murata Electronics
- C2: DIS (none) -> DigiKey; DPN (none) -> 490-GRT188R71E105KE13DCT-ND; MPN (none) -> GRT188R71E105KE13D; Manufacturer (none) -> Murata Electronics

Commit message: Revert "Merge branch 'master' of github.com:psas/lv3.1-avionics"
This reverts commit e8b3300ae824ca3338ac8ec8f922a1d509083487, reversing
changes made to 8f716272e32ab4533c36fe5f3d4033526be42e02.
Parts:
- C1, C3, C4, C5: footprint CameraBoard:.0805-B-NOSILK -> oresat-passives:0805-C-NOSILK; DIS DigiKey -> Digikey; Manufacturer Murata Electronics -> (none); Manufacturer_Name (none) -> Murata Electronics
- C10: footprint Capacitor_SMD:C_0603_1608Metric -> oresat-passives:0603-C-NOSILK; DIS (none) -> Digikey; DPN (none) -> 490-GRT188R71E105KE13DCT-ND; MPN (none) -> GRT188R71E105KE13D; Manufacturer_Name (none) -> Murata Electronics
- C11, C12, C9: footprint CameraBoard:1206-A -> oresat-passives:1206-C; DIS (none) -> Digikey; DPN (none) -> 490-5528-1-ND; MPN (none) -> GRM31CR61A476ME15L; Manufacturer_Name (none) -> Murata Electronics
- C13: footprint Capacitor_SMD:C_1206_3216Metric -> oresat-passives:1206-C; DIS (none) -> Digikey; DPN (none) -> 445-12883-1-ND; MPN (none) -> CGA5L3X5R1H106M160AB; Manufacturer_Name (none) -> TDK
- C2: footprint Capacitor_SMD:C_0805_2012Metric -> oresat-passives:0805-C-NOSILK; DIS DigiKey -> Digikey; DPN 490-GRT188R71E105KE13DCT-ND -> 490-10675-2-ND; MPN GRT188R71E105KE13D -> GCM21BR71H105KA03L; Manufacturer Murata Electronics -> (none); Manufacturer_Name (none) -> Murata Electronics
- C6: footprint Capacitor_SMD:C_1206_3216Metric -> oresat-passives:1206-C; DIS (none) -> Digikey; DPN (none) -> 1276-1072-1-ND; MPN (none) -> CL31B225KAHNNNE; Manufacturer_Name (none) -> Samsung Electro-Mechanics
- C7: footprint CameraBoard:.0603-A-NOSILK -> oresat-passives:0603-C-NOSILK; DIS (none) -> Digikey; DPN (none) -> 399-12983-1-ND; MPN (none) -> C0603C103J5RACAUTO; Manufacturer_Name (none) -> KEMET
- C8: footprint Capacitor_SMD:C_0603_1608Metric -> oresat-passives:0603-C-NOSILK; DIS (none) -> Digikey; DPN (none) -> 399-6856-1-ND; MPN (none) -> C0603C104K5RACAUTO; Manufacturer_Name (none) -> KEMET
- D2, D3, D5: footprint LED_SMD:LED_0603_1608Metric -> oresat-diodes:LED_0603_1608Metric; DIS (none) -> Digikey; DPN (none) -> 732-150060AS75000CT-ND; MPN (none) -> 150060AS75000; Manufacturer_Name (none) -> Wurth
- D4: DIS (none) -> Digikey; DPN (none) -> MBRS340T3GOSCT-ND; MPN (none) -> MBRS340T3G; Manufacturer_Name (none) -> onsemi
- D6: DIS (none) -> Digikey; DPN (none) -> B240A-FDICT-ND; MPN (none) -> B240A-13-F; Manufacturer_Name (none) -> Diodes Incorporated
- JP1, JP2, JP3: DIS (none) -> Digikey; DPN (none) -> 732-5315-ND; MPN (none) -> 61300211121; Manufacturer_Name (none) -> Würth Elektronik
- JP10, JP11, JP12, JP13, JP14, JP5, JP6, JP7, JP8, JP9: DIS (none) -> Digikey; DPN (none) -> 732-5316-ND; MPN (none) -> 61300311121; Manufacturer_Name (none) -> Würth Elektronik
- JP4: DIS (none) -> Digikey; DPN (none) -> 732-5319-ND; MPN (none) -> 61300611121; Manufacturer_Name (none) -> Würth Elektronik
- L1: DIS (none) -> Digikey; DPN (none) -> 732-6785-1-ND; MPN (none) -> 74477110; Manufacturer_Name (none) -> Würth Elektronik
- L2: footprint Inductor_SMD:L_0603_1608Metric -> oresat-misc:WE-PD_1260; DIS (none) -> Digikey; DPN (none) -> 732-1208-1-ND; MPN (none) -> 74477110; Manufacturer_Name (none) -> Würth Elektronik
- Q1, Q2, Q3: DIS (none) -> Digikey; DPN (none) -> SUD08P06-155L-GE3CT-ND; MPN (none) -> SUD08P06-155L-GE3; Manufacturer_Name (none) -> Vishay Siliconix
- R1, R2, R4, R6: footprint Resistor_SMD:R_0603_1608Metric -> oresat-passives:0603-C-NOSILK; DIS (none) -> Digikey; DPN (none) -> RMCF0603FT10K0CT-ND; MPN (none) -> RMCF0603FT10K0; Manufacturer_Name (none) -> Stackpole Electronics
- R10: footprint Resistor_SMD:R_0603_1608Metric -> oresat-passives:0603-C-NOSILK; DIS (none) -> Mouser; DPN (none) -> 71-TNPW060338K8BEEA; MPN (none) -> TNPW060338K8BEEA; Manufacturer_Name (none) -> Vishay
- R11, R12: footprint Resistor_SMD:R_0603_1608Metric -> oresat-passives:0603-C-NOSILK; DIS (none) -> Digikey; DPN (none) -> RMCF0603FT2K70CT-ND; MPN (none) -> RMCF0603FT1K00; Manufacturer_Name (none) -> Stackpole Electronics Inc
- R13: footprint Resistor_SMD:R_0603_1608Metric -> oresat-passives:0603-C-NOSILK; DIS (none) -> Digikey; DPN (none) -> 541-3.30KHCT-ND; MPN (none) -> CRCW06033K30FKEA; Manufacturer_Name (none) -> Vishay Dale
- R14: footprint Resistor_SMD:R_0603_1608Metric -> oresat-passives:0603-C-NOSILK; DIS (none) -> Digikey; DPN (none) -> 13-RC0603FR-10150KLCT-ND; MPN (none) -> RC0603FR-10150KL; Manufacturer_Name (none) -> YAEGO
- R3: footprint Resistor_SMD:R_0603_1608Metric -> oresat-passives:0603-C-NOSILK; DIS (none) -> Digikey; DPN (none) -> 541-133KHCT-ND; MPN (none) -> CRCW0603133KFKEA; Manufacturer_Name (none) -> Vishay Dale
- R5: footprint Resistor_SMD:R_0603_1608Metric -> oresat-passives:0603-C-NOSILK; DIS (none) -> Digikey; DPN (none) -> RMCF0603FT33K0CT-ND; MPN (none) -> RMCF0603FT33K0; Manufacturer_Name (none) -> Stackpole Electronics
- R7: footprint Resistor_SMD:R_0603_1608Metric -> oresat-passives:0603-C-NOSILK; DIS (none) -> Digikey; DPN (none) -> P2.00KHCT-ND; MPN (none) -> ERJ-3EKF2001V; Manufacturer_Name (none) -> Panasonic Industry
- R8: footprint Resistor_SMD:R_0603_1608Metric -> oresat-passives:0603-C-NOSILK; DIS (none) -> Digikey; DPN (none) -> RMCF0603FT3K00CT-ND; MPN (none) -> RMCF0603FT3K00; Manufacturer_Name (none) -> Stackpole Electronics Inc
- R9: footprint Resistor_SMD:R_0603_1608Metric -> oresat-passives:0603-C-NOSILK; DIS (none) -> Digikey; DPN (none) -> MCT06030D6501BP100-ND; MPN (none) -> MCT06030D6501BP100; Manufacturer_Name (none) -> Vishay
- TH1: footprint Resistor_SMD:R_0603_1608Metric -> oresat-misc:THRMC1608X95N; DIS (none) -> Digikey; DPN (none) -> 490-16279-1-ND; MPN (none) -> NCU18XH103F60RB; Manufacturer_Name (none) -> Murata Electronics
- TP1, TP2, TP3: DIS (none) -> Digikey; now left out of the parts list
- U1: DIS (none) -> Digikey; DPN (none) -> LM2678S-ADJ/NOPB-ND; MPN (none) -> LM2678S-ADJ/NOPB; Manufacturer_Name (none) -> Texas Instruments
- U2: DIS (none) -> Digikey; DPN (none) -> 1589-MP2659GQ-0000-ZCT-ND; MPN (none) -> MP2659GQ-0000-Z
