File: CameraBoard/kicad/CameraBoard.kicad_pcb (KiCad board)
At the start: 2 copper layers, 101.6 x 76.2 mm, 57 parts, among them Q1 SUD08P06-155L, Q2 SUD08P06-155L, Q3 SUD08P06-155L, U1 MP2659GQ-0000-Z

Commit message: Minor layout changes
Routing:
- net +12V: track 408.9 -> 353.3 mm
- net GND: track 11.5 -> 7.15 mm, vias 119 -> 120
- net Net-(Q2-S): track 27.7 -> 25.6 mm
Changed lines of the file:
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@@
 	)
 	(segment
-		(start 137.4 117.35)
-		(end 137.3 117.45)
-		(width 0.7)
-		(layer "F.Cu")
-		(net "+12V")
-	)
-	(segment
 		(start 102.7 114.1)
 		(end 100.0511 114.1)
@@
 	)
 	(segment
-		(start 136.25 117.45)
-		(end 137.3 117.45)
-		(width 0.7)
-		(layer "F.Cu")
-		(net "+12V")
-	)
-	(segment
 		(start 193.2 102.56)
 		(end 195.9411 102.56)
@@
 	)
 	(segment
-		(start 106.9 117)
-		(end 106.9 108.54)
-		(width 1)
-		(layer "F.Cu")
-		(net "+12V")
-	)
-	(segment
 		(start 99.9511 127.5436)
 		(end 99.9511 130.1036)
@@
 	)
 	(segment
-		(start 99.9911 108.64)
-		(end 99.9511 108.6)
-		(width 0.2)
-		(layer "F.Cu")
-		(net "+12V")
-	)
-	(segment
 		(start 196.2011 130.8536)
 		(end 185.6977 141.357)
@@
 	)
 	(segment
-		(start 107.4 117.5)
-		(end 106.9 117)
-		(width 1)
-		(layer "F.Cu")
-		(net "+12V")
-	)
-	(segment
 		(start 123.0411 141.3536)
 		(end 111.2011 141.3536)
@@
 	)
 	(segment
-		(start 137.4 104.8)
-		(end 137.4 117.35)
-		(width 0.7)
-		(layer "F.Cu")
-		(net "+12V")
-	)
-	(segment
 		(start 99.9511 108.6)
 		(end 99.9511 87.5436)
@@
 	)
 	(segment
-		(start 136.2 117.5)
-		(end 136.25 117.45)
-		(width 0.7)
-		(layer "F.Cu")
-		(net "+12V")
-	)
-	(segment
 		(start 99.9511 127.5436)
 		(end 99.9511 116.7)
@@
 	)
 	(segment
-		(start 128.25 117.5)
-		(end 136.2 117.5)
-		(width 0.95)
-		(layer "F.Cu")
-		(net "+12V")
-	)
-	(segment
 		(start 99.9511 114.2)
 		(end 99.9511 108.6)
@@
 	)
 	(segment
-		(start 102.9 108.54)
-		(end 106.9 108.54)
-		(width 1.000001)
-		(layer "F.Cu")
-		(net "+12V")
-	)
-	(segment
 		(start 151.2011 141.3536)
 		(end 151.2011 139.2611)
@@
 	)
 	(segment
-		(start 128.25 117.5)
-		(end 107.4 117.5)
-		(width 1)
-		(layer "F.Cu")
-		(net "+12V")
-	)
-	(segment
-		(start 102.7 108.64)
-		(end 99.9911 108.64)
+		(start 128.3 141.3536)
+		(end 123.0411 141.3536)
 		(width 1.6)
 		(layer "F.Cu")
@@
 	)
 	(segment
-		(start 128.3 141.3536)
-		(end 123.0411 141.3536)
+		(start 151.2011 141.3536)
+		(end 142.1 141.3536)
 		(width 1.6)
 		(layer "F.Cu")
@@
 	)
 	(segment
-		(start 151.2011 141.3536)
-		(end 142.1 141.3536)
+		(start 102.9 108.54)
+		(end 100.0111 108.54)
 		(width 1.6)
 		(layer "F.Cu")
@@
 	)
 	(segment
-		(start 175.35 87.91875)
-		(end 175.35 87.51875)
+		(start 138.1 123.2)
+		(end 138.1 122.05)
 		(width 0.2)
 		(layer "F.Cu")
@@
 	)
 	(segment
-		(start 174.3 83.7)
-		(end 175.1 83.7)
+		(start 137.8 123.5)
+		(end 138.1 123.2)
 		(width 0.2)
 		(layer "F.Cu")
@@
 	)
 	(segment
-		(start 175.35 87.51875)
-		(end 177.68125 87.51875)
+		(start 174.3 83.7)
+		(end 175.1 83.7)
 		(width 0.2)
 		(layer "F.Cu")
@@
 	)
 	(segment
-		(start 175.35 87.11875)
-		(end 175.35 87.51875)
+		(start 175.35 87.51875)
+		(end 177.68125 87.51875)
 		(width 0.2)
 		(layer "F.Cu")
@@
 	)
 	(segment
-		(start 125.74 70.7)
-		(end 128.28 70.7)
-		(width 0.2)
-		(layer "F.Cu")
-		(net "GND")
-	)
-	(segment
-		(start 128.28 70.7)
-		(end 130.82 70.7)
-		(width 0.2)
-		(layer "F.Cu")
-		(net "GND")
-	)
-	(segment
 		(start 173.75 85.91875)
 		(end 173.75 84.25)
@@
 	)
 	(via
+		(at 173.9 86.9)
+		(size 0.6)
+		(drill 0.3)
+		(layers "F.Cu" "B.Cu")
+		(free yes)
+		(net "GND")
+	)
+	(via
 		(at 133.95 74.35)
 		(size 0.6)
@@
 	)
 	(via
-		(at 137.2 123.575)
+		(at 137.8 123.5)
 		(size 0.6)
 		(drill 0.3)
@@
 	)
 	(via
-		(at 102.925 117.925)
+		(at 105.6 114.4)
 		(size 0.604)
 		(drill 0.35)
@@
 	)
 	(segment
-		(start 170.3 98.5)
-		(end 164.2 98.5)
-		(width 0.7)
-		(layer "F.Cu")
-		(net "/VUMB")
-	)
-	(segment
 		(start 163.65 82.4)
 		(end 163.635 82.385)
@@
 	(segment
 		(start 170.3 98.5)
-		(end 170.3 93.564461)
-		(width 0.6)
+		(end 164.2 98.5)
+		(width 0.7)
 		(layer "F.Cu")
 		(net "/VUMB")
 	)
 	(segment
-		(start 164.2 98.5)
-		(end 163.65 97.95)
-		(width 0.7)
+		(start 170.3 93.564461)
+		(end 173.35 90.514461)
+		(width 0.6)
 		(layer "F.Cu")
 		(net "/VUMB")
@@
 	)
 	(segment
-		(start 173.4 88.26875)
-		(end 173.4 90)
-		(width 0.25)
+		(start 163.65 97.95)
+		(end 163.65 92.4)
+		(width 0.7)
 		(layer "F.Cu")
 		(net "/VUMB")
 	)
 	(segment
-		(start 163.65 97.95)
-		(end 163.65 92.4)
+		(start 164.2 98.5)
+		(end 163.65 97.95)
 		(width 0.7)
 		(layer "F.Cu")
@@
 	)
 	(segment
+		(start 173.4 88.26875)
+		(end 173.4 90)
+		(width 0.25)
+		(layer "F.Cu")
+		(net "/VUMB")
+	)
+	(segment
 		(start 163.65 92.4)
 		(end 163.65 85.7)
@@
 	)
 	(segment
-		(start 170.3 93.564461)
-		(end 173.35 90.514461)
-		(width 0.6)
+		(start 170.375 98.575)
+		(end 170.375 100.355)
+		(width 0.2)
 		(layer "F.Cu")
 		(net "/VUMB")
 	)
 	(segment
-		(start 170.375 98.575)
-		(end 170.375 100.355)
-		(width 0.2)
+		(start 170.3 98.5)
+		(end 170.3 93.564461)
+		(width 0.6)
 		(layer "F.Cu")
 		(net "/VUMB")
@@
 	)
 	(segment
-		(start 134.8 115)
-		(end 133.4 115)
+		(start 132.22 98.82)
+		(end 129.34 98.82)
 		(width 1)
 		(layer "F.Cu")
@@
 	)
 	(segment
-		(start 133 114.6)
-		(end 133 99.6)
+		(start 133 99.6)
+		(end 132.22 98.82)
 		(width 1)
 		(layer "F.Cu")
@@
 	)
 	(segment
-		(start 133 99.6)
-		(end 132.22 98.82)
+		(start 133 108.2)
+		(end 133 106.3)
 		(width 1)
 		(layer "F.Cu")
@@
 	)
 	(segment
-		(start 134.8 115)
-		(end 136.2 115)
-		(width 1)
-		(layer "F.Cu")
-		(net "Net-(Q2-S)")
-	)
-	(segment
-		(start 132.22 98.82)
-		(end 129.34 98.82)
-		(width 1)
-		(layer "F.Cu")
-		(net "Net-(Q2-S)")
-	)
-	(segment
-		(start 133.4 115)
-		(end 133 114.6)
+		(start 133 106.3)
+		(end 133 99.6)
 		(width 1)
 		(layer "F.Cu")
@@
 	)
 	(via
-		(at 136.2 115)
+		(at 133 108.2)
 		(size 0.9)
 		(drill 0.6)
@@
 	)
 	(via
-		(at 134.8 115)
+		(at 133 106.3)
 		(size 0.9)
 		(drill 0.6)
@@
 	)
 	(segment
-		(start 134.8 115)
+		(start 133 110)
+		(end 138 115)
+		(width 1)
+		(layer "B.Cu")
+		(net "Net-(Q2-S)")
+	)
+	(segment
+		(start 133 106.3)
+		(end 133 110)
+		(width 1)
+		(layer "B.Cu")
+		(net "Net-(Q2-S)")
+	)
+	(segment
+		(start 138 115)
 		(end 139.4 115)
 		(width 1)
@@
 		(polygon
 			(pts
-				(xy 137.8 118) (xy 137.8 108.5) (xy 141.2 108.5) (xy 141.2 99.9) (xy 133.85 99.9) (xy 133.9 108.35)
-				(xy 133.9 115.7) (xy 109.45 115.6) (xy 109.5 107.25) (xy 100.449996 107.199722) (xy 100.425485 112.25)
-				(xy 103.8 112.25) (xy 103.75 120.45) (xy 128.5 120.45) (xy 128.5 119.05) (xy 136.85 119.2) (xy 136.9 118)
+				(xy 137.727562 118.006306) (xy 137.733817 108.49772) (xy 139.1 108.498619) (xy 139.1 99.9) (xy 133.85 99.9)
+				(xy 133.9 108.35) (xy 133.9 115.7) (xy 99.698127 115.726998) (xy 99.701872 120.471622) (xy 128.504339 120.507335)
+				(xy 128.498086 119.245291) (xy 136.90778 119.190323) (xy 136.9 118)
 			)
 		)
@@
 	)
 	(zone
-		(net "GND")
-		(layer "F.Cu")
-		(hatch edge 0.5)
-		(priority 1)
-		(connect_pads
-			(clearance 0.2)
-		)
-		(min_thickness 0.127)
-		(fill yes
-			(thermal_gap 0.127)
-			(thermal_bridge_width 0.5)
-			(smoothing fillet)
-			(radius 0.2)
-			(island_removal_mode 0)
-		)
-		(polygon
-			(pts
-				(xy 199.3773 143.1798) (xy 97.62485 143.1798) (xy 97.67495 66.8274) (xy 199.3773 66.8274)
-			)
-		)
-	)
-	(zone
 		(net "/BATT+")
 		(layer "F.Cu")
@@
 		(hatch edge 0.5)
 		(priority 2)
-		(connect_pads
+		(connect_pads yes
 			(clearance 0.2)
 		)
@@
 		(polygon
 			(pts
-				(xy 170.8 84.1) (xy 170.8 90.5) (xy 177.1 90.5) (xy 177.1 84.1)
+				(xy 170.8 84.1) (xy 170.8 86.4) (xy 173 86.4) (xy 173 84.1)
 			)
 		)
@@
 	)
 	(zone
+		(net "GND")
+		(locked yes)
+		(layers "F.Cu" "B.Cu")
+		(hatch edge 0.5)
+		(priority 1)
+		(connect_pads
+			(clearance 0.2)
+		)
+		(min_thickness 0.127)
+		(fill yes
+			(thermal_gap 0.127)
+			(thermal_bridge_width 0.5)
+			(smoothing fillet)
+			(radius 0.2)
+			(island_removal_mode 0)
+		)
+		(polygon
+			(pts
+				(xy 199.3773 143.1798) (xy 97.62485 143.1798) (xy 97.67495 66.8274) (xy 199.3773 66.8274)
+			)
+		)
+	)
+	(zone
 		(layer "B.Cu")
 		(hatch edge 0.5)
@@
 	(zone
 		(net "GND")
+		(locked yes)
 		(layer "B.Cu")
 		(hatch edge 0.5)

Commit message: Schematic and PCB Changes
-Added symbols and footprints to library
-Changed a couple mosfets and the thermistor for better fits
-Added more description to connectors
-Added power flags
-Edited IC symbols to match datasheets
-Made sure all components had values showing
-Added descriptive names to connectors on PCB
-Rearranged PCB after switching out some components footprints
Parts:
- added TP10: Test-Point, oresat-misc:TestPoint-0.75mm-th, F.Cu at (118.6, 138.5)
- added TP11: Test-Point, oresat-misc:TestPoint-0.75mm-th, F.Cu at (182.7, 71.1)
- added TP4: Test-Point, oresat-misc:TestPoint-0.75mm-th, F.Cu at (193.2, 111.6)
- added TP5: Test-Point, oresat-misc:TestPoint-0.75mm-th, F.Cu at (141.4, 138.7)
- added TP6: Test-Point, oresat-misc:TestPoint-0.75mm-th, F.Cu at (102.8, 119.4)
- added TP7: Test-Point, oresat-misc:TestPoint-0.75mm-th, F.Cu at (193.5, 90.4)
- added TP8: Test-Point, oresat-misc:TestPoint-0.75mm-th, F.Cu at (193.4, 130.8)
- added TP9: Test-Point, oresat-misc:TestPoint-0.75mm-th, F.Cu at (169.0, 138.6)
- D4: value D_MBRS340T3G -> VS-6TQ045S-M3; footprint Diode_SMD:D_SMC -> oresat-diodes:VS6TQ045SM3
- D5: value LED_Small_Filled -> GRN
- L1: value 784770220 -> 22uh; footprint CameraBoard:784770220 -> Inductor_SMD:L_Vishay_IHLP-4040
- Q1: value SUD08P06-155L -> DMG3404L-7; footprint Package_TO_SOT_SMD:TO-252-2 -> oresat-transistors:DMG3404L_DIO
- Q3: value SUD08P06-155L -> AOD4185; footprint Package_TO_SOT_SMD:TO-252-2 -> oresat-transistors:TO252_AOS-M
- R13: value 3.3k -> 10k
- TH1: footprint oresat-misc:THRMC1608X95N -> Resistor_THT:R_Axial_DIN0204_L3.6mm_D1.6mm_P2.54mm_Vertical
- TP1, TP2, TP3: footprint CameraBoard:2MM-TEST-POINT -> oresat-misc:TestPoint-0.75mm-th
- U2: value ~ -> LM2678SD-ADJ/NOPB; footprint CameraBoard:LM2678SD-12_NOPB -> psas-footprints:SRC14A
- moved R2 29.6 mm to (130.6, 88.2), turned to 180 degrees
- moved JP1 25.8 mm to (133.8, 91.0), turned to -90 degrees
- moved Q1 17.8 mm to (130.3, 95.0), turned to 180 degrees
- moved TP1 7.07 mm to (133.2, 116.8)
- moved D4 6.88 mm to (133.0, 124.2), turned to -90 degrees
- moved R1 6.57 mm to (123.0, 100.0), turned to -90 degrees
- moved C1 6.02 mm to (143.1, 106.7)
- moved C11 6.02 mm to (132.0, 112.9)
- moved C3 6.02 mm to (145.0, 106.7)
- moved C5 6.02 mm to (141.2, 106.7)
- moved C7 6.02 mm to (144.1, 113.5)
- moved C9 6.02 mm to (129.5, 112.9)
- moved L1 6.02 mm to (142.0, 98.8), turned to 180 degrees
- moved C12 6.02 mm to (134.4, 112.9)
- moved C4 6.02 mm to (139.3, 106.7)
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Connections:
- C1 pad 1: Net-(Q2-S) -> Net-(Q2-D)
- C3 pad 1: Net-(Q2-S) -> Net-(Q2-D)
- C4 pad 1: Net-(Q2-S) -> Net-(Q2-D)
- C5 pad 1: Net-(Q2-S) -> Net-(Q2-D)
- C7 pad 1: /SOUT -> Net-(D4-K)
- D4 pad 1: /SOUT -> unconnected-(D4-NC-Pad1)
- D4 pad 2: GND -> Net-(D4-K)
- JP10 pad 3: unconnected-(JP10-Pin_3-Pad3) -> Net-(JP10-Pin_3)
- JP11 pad 3: unconnected-(JP11-Pin_3-Pad3) -> Net-(JP11-Pin_3)
- JP12 pad 3: unconnected-(JP12-Pin_3-Pad3) -> Net-(JP12-Pin_3)
- JP13 pad 3: unconnected-(JP13-Pin_3-Pad3) -> Net-(JP13-Pin_3)
- JP6 pad 3: unconnected-(JP6-Pin_3-Pad3) -> Net-(JP6-Pin_3)
- JP7 pad 3: unconnected-(JP7-Pin_3-Pad3) -> Net-(JP7-Pin_3)
- JP8 pad 3: unconnected-(JP8-Pin_3-Pad3) -> Net-(JP8-Pin_3)
- JP9 pad 3: unconnected-(JP9-Pin_3-Pad3) -> Net-(JP9-Pin_3)
- L1 pad 1: /SOUT -> Net-(D4-K)
- Q1 pad 2: Net-(Q1-D) -> GND
- Q1 pad 3: GND -> Net-(Q1-D)
- Q2 pad 2: VBATT -> Net-(Q2-D)
- Q2 pad 3: Net-(Q2-S) -> VBATT
- U2 pad 12: /SOUT -> Net-(D4-K)
- U2 pad 13: /SOUT -> Net-(D4-K)
- U2 pad 14: /SOUT -> Net-(D4-K)
- U2 pad 2: Net-(Q2-S) -> Net-(Q2-D)
- U2 pad 3: Net-(Q2-S) -> Net-(Q2-D)
Routing:
- net Net-(D4-K): track 0.00 -> 30.3 mm
- net /SOUT: track 30.3 -> 0.00 mm
- net Net-(Q2-S): track 25.6 -> 0.00 mm, vias 4 -> 0
- net Net-(Q2-D): track 0.00 -> 14.2 mm, vias 0 -> 4
- net VBATT: track 15.2 -> 9.32 mm
- net Net-(JP11-Pin_3): track 0.00 -> 4.99 mm
- net Net-(JP12-Pin_3): track 0.00 -> 4.72 mm
- net Net-(JP7-Pin_3): track 0.00 -> 4.71 mm
- net Net-(JP6-Pin_3): track 0.00 -> 3.98 mm
- net Net-(JP13-Pin_3): track 0.00 -> 3.67 mm
- net Net-(JP10-Pin_3): track 0.00 -> 3.26 mm
- net Net-(JP1-Pin_2): track 8.83 -> 5.64 mm
- net Net-(JP8-Pin_3): track 0.00 -> 3.05 mm
- net Net-(JP9-Pin_3): track 0.00 -> 2.91 mm
- net +12V: track 353.3 -> 355.2 mm
- added copper zone on F.Cu, net Net-(D4-K)
- added copper zone on F.Cu, net Net-(Q2-D)
- removed copper zone on F.Cu, net /SOUT
- removed copper zone on F.Cu, net Net-(Q2-S)
Other:
- board text added: "ARM"
- board text added: "ARM In"
- board text added: "ARM Out"
- board text added: "BATTERY"
- board text added: "CAM"
- board text added: "CAM DOWN"
- board text added: "To Vumb"
- board text removed: "ARM+"
- board text removed: "ARM-"
- board text removed: "Cam Up"

Commit message: Small PCB Updates
-Added more ground vias
-Moved capacitor closer to IC
-Moved TP3 closer to track
Parts:
- moved C13 42.3 mm to (166.6, 81.3), turned to 90 degrees
- moved TP3 5.48 mm to (158.8, 86.9)
- moved R5 0.52 mm to (165.4, 86.7)
Routing:
- net GND: track 7.43 -> 1.86 mm, vias 120 -> 134
- net /BATT+: track 98.8 -> 94.9 mm
- net Net-(D1-K): track 19.6 -> 18.9 mm
- net Net-(U1-ILIM): track 7.79 -> 8.41 mm

Commit message: Camerca board v2.0 off to fab
Pretty-ified schematic by moving things around and redoing the switching supply symbol. Moved labels around, made them all 1.27 mm.
Fixed BOM by collapsing Rs and Cs together, and brought them up to speed with OReSat shared BOM list. Added tons more capacitance
to the SPS because of the datasheets claiming it was important. Moved RocketReady connector to board edge, like other connectors.
Parts:
- added C14: 1u, oresat-passives:0805-C-NOSILK, F.Cu at (145.0, 110.1)
- added C15: 100u, Capacitor_SMD:CP_Elec_8x10.5, F.Cu at (121.3, 115.9)
- added C16: 100u, Capacitor_SMD:CP_Elec_8x10.5, F.Cu at (111.9, 115.9)
- C1, C3, C4, C5: footprint oresat-passives:0805-C-NOSILK -> oresat-passives:1206-C
- C10: footprint oresat-passives:0603-C-NOSILK -> oresat-passives:0805-C-NOSILK
- C11, C12, C9: value 47u -> 10u
- D2, D3: value LED_Small_Filled -> AMB
- D4: value VS-6TQ045S-M3 -> MBRD835; footprint oresat-diodes:VS6TQ045SM3 -> Package_TO_SOT_SMD:TO-252-2
- L1: value 22uh -> 22u
- L2: value 10uh -> 10u
- Q2: value SUD08P06-155L -> AOD4185; footprint Package_TO_SOT_SMD:TO-252-2 -> oresat-transistors:TO252_AOS-M
- R10: value 38.4k -> 38.3k
- R9: value 6.95k -> 6.98k
- moved JP1 21.5 mm to (142.0, 71.2)
- moved D4 6.39 mm to (139.4, 123.6)
- moved R1 5.51 mm to (128.0, 97.7), turned to 0 degrees
- moved R2 4.00 mm to (130.1, 92.2), turned to 0 degrees
- moved TP1 1.86 mm to (135.0, 117.3)
- moved C4 0.70 mm to (138.6, 106.7)
- moved C5 0.45 mm to (140.8, 106.7)
- moved C1 0.20 mm to (142.9, 106.7)
- moved Q1 0.15 mm to (130.3, 94.8), turned to -90 degrees
- turned Q2 to 180 degrees
Connections:
- U2 pad 15: (no net) -> GND
Routing:
- net Net-(JP1-Pin_2): track 5.64 -> 27.0 mm, vias 0 -> 2
- net Net-(Q2-D): track 14.2 -> 0.00 mm, vias 4 -> 14
- net Net-(D4-K): track 30.3 -> 20.0 mm
- net Net-(Q1-D): track 12.1 -> 7.02 mm
- net Net-(U2-ON): track 4.05 -> 2.50 mm
- net GND: track 1.86 -> 0.70 mm, vias 134 -> 150
- net VBATT: track 9.32 -> 10.3 mm
- added copper zone on B.Cu, net Net-(Q2-D)
Other:
- board text added: "${TITLE} v${REVISION} ${ISSUE_DATE}"
- board text added: "CAM DWN"
- board text added: "RR"
- board text removed: "12V at 5A max"
- board text removed: "16.8V to 12V SPS"
- board text removed: "19V at 2.5A charge current"
- board text removed: "Battery Charger"
- board text removed: "CAM DOWN"
- board text removed: "Camera Board Rev 2.0 ${CURRENT_DATE}"
