File: WiringDiagram/WiringDiagram.kicad_sch (KiCad schematic)
At the start: 56 parts, among them J1 Conn_01x06, J2 Conn_01x02, J3 Conn_01x04, J4 Conn_01x04, J5 Conn_01x06, J6 Conn_01x08, J7 Conn_01x04, J8 FTDI SERIAL, J9 Conn_01x04, SW1 TELEMETRUM ROTARY SWITCH, SW2 ERS SENDER ROTARY SWITCH, SW3 CAMERA BOARD ROTARY SWITCH

Commit message: Updated wiring diagram for upcoming LV3.1  Launch 15 flight
Parts:
- removed CAM-J9: BATTERY, symbol Connector_Generic:Conn_01x06
- removed CAM-JP10: ATV TX, symbol Connector_Generic:Conn_01x03
- removed ERS-J13, ERS-J16, ERS-J17, ERS-J9: SERIAL, symbol Connector_Generic:Conn_01x03
- removed J8: FTDI SERIAL, symbol Connector_Audio:AudioJack2_Ground
- added BT3: 9V battery, symbol Device:Battery_Cell
- added CAM-JP13: CAMERA, symbol Connector_Generic:Conn_01x03
- added CAM-JP2: ARM, symbol Connector_Generic:Conn_01x02
- added CAM-JP3: UMB, symbol Connector_Generic:Conn_01x02
- added J10, J11, J12, J8: Conn_01x04, symbol Connector_Generic:Conn_01x04
- added SW4: PERFECTFLITE FLIGHT COMPUTER, symbol Switch:SW_SPST
- BT1: value Battery_Cell -> LiPo Cell
- CAM-JP1: renamed from CAM-JP8; value Thermistor -> RocketReady
- CAM-JP10: renamed from CAM-JP2; value ~ -> CAMERA
- CAM-JP11: renamed from ERS-J23; value SERIAL -> CAMERA
- CAM-JP12: renamed from ERS-J21; value SERIAL -> CAMERA
- CAM-JP14: renamed from CAM-JP1; value ~ -> ATV TX
- CAM-JP5: renamed from ERS-J19; value SERIAL -> CAMERA DWN
- CAM-JP7: renamed from ERS-J22; value SERIAL -> CAMERA
- CAM-JP8: renamed from ERS-J20; value SERIAL -> CAMERA
- renumbered CAM-J11 to CAM-JP4, CAM-JP12 to CAM-JP6, CAM-JP13 to CAM-JP9
Connections:
- net 5V is gone; now on net 12V: ERS-J14.3 (Pin_3), ERS-J15.3 (Pin_3), J5.6 (Pin_6)
- net ARM+: now also CAM-JP2.2 (Pin_2)
- net ARM-: now also CAM-JP2.1 (Pin_1)
- net GND: now also CAM-JP1.1 (Pin_1), CAM-JP14.2 (Pin_2), CAM-JP3.1 (Pin_1), CAM-JP3.2 (Pin_2); no longer CAM-JP1.2 (Pin_2)
- net VIDEO: now also CAM-JP14.3 (Pin_3)
- net 12V: now reaches CAM-JP14.1 (Pin_1)
- net at ERS-J5.1 (Pin_1), J9.2 (Pin_2): now also CAM-JP1.2 (Pin_2)
- new net: BT3.1 (+), J11.1 (Pin_1)
- new net: BT3.2 (-), J11.2 (Pin_2)
- new net: J11.3 (Pin_3), J8.1 (Pin_1), J8.2 (Pin_2)
- new net: J11.4 (Pin_4), J8.3 (Pin_3), J8.4 (Pin_4)
- new net: J10.3 (Pin_3), J10.4 (Pin_4), SW4.1 (A)
- new net: J10.1 (Pin_1), J10.2 (Pin_2), SW4.2 (B)
- no-connect marks 7 -> 6
Other:
- note added: ""A""
- note added: ""B"/Red"
- note added: ""Combiner""
- note added: "6 in"
- note added: "CAMERA MODULE"
- note added: "DOWN FRONT"
- note added: "DOWN LEFT"
- note added: "DOWN RIGHT"
- note added: "PerfectFlite"
- note added: "Switch closed = On"
- note added: "UPPER CAMERA MODULE"
- note removed: "CAMERA"
- note removed: "CHECK TX/RX NOT CHECKED!!"
- note removed: "GND connection for VUMB :("
- note removed: "TO FRONT CAMERA FACING DOWN"
- note removed: "TO FRONT CAMERA FACING UP"
- note removed: "TO VIDEO TX"
- note removed: "UMB"
- title: LV3.1 Avionics Module Wiring Diagram -> LV3.1 L15 Avionics Module Wiring Diagram
- moved on the sheet: AE1, AE2, BT1, BT2, CAM-B1, CAM-JP1, CAM-JP10, CAM-JP14, CAM-JP4, CAM-JP6, CAM-JP9, ERS-J10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

Commit message: Add alphabetical connector and numerical wire labels
Connections:
- net GND: now also ERS-J5.2 (Pin_2), J9.3 (Pin_3)
- net RR: now also CAM-JP1.2 (Pin_2), ERS-J5.1 (Pin_1), J9.2 (Pin_2)
Other:
- note added: ""1""
- note added: ""10""
- note added: ""11""
- note added: ""12""
- note added: ""13""
- note added: ""14""
- note added: ""16""
- note added: ""17""
- note added: ""18""
- note added: ""19""
- note added: ""2""
- note added: ""20""
- note added: ""3""
- note added: ""4""
- note added: ""5""
- note added: ""6""
- note added: ""7""
- note added: ""8""
- note added: ""9""
- note added: ""C""
- note added: ""D""
- note added: ""E""
- note added: ""F""
- note added: ""G""
- note added: ""H""
- note added: ""I""
- note added: ""J""
- note added: ""K""
- note added: ""L""
